File: Hardware/Mini-Esp/R2/Sandy R2.brd (EAGLE design)
At the start: 25.7 x 23 mm, 18 parts, among them SW1 RST, SW2 PR

Commit message: Update Mini-Esp and SwitchNode R2
Parts:
- SW2: value PR -> FLASH
Other:
- board size 25.7 x 23 mm -> 25.7 x 24.6 mm
- board text added: "#0"
- board text added: "#2"
- board text added: "#4"
- board text added: "#5"
- board text added: "Flash"
- board text removed: "0"
- board text removed: "2"
- board text removed: "4"
- board text removed: "5"
- board text removed: "G"
