File: Hardware/Mini-Esp/R2/Sandy R2.sch (EAGLE design)
At the start: 18 parts, among them SW1 RST, SW2 PR

Commit message: Update Mini-Esp and SwitchNode R2
Parts:
- SW2: value PR -> FLASH
Changed lines of the file:
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@@
 <part name="GND6" library="SparkFun" deviceset="GND" device=""/>
 <part name="SW1" library="MySMD" deviceset="PB157" device="" value="RST"/>
-<part name="SW2" library="MySMD" deviceset="PB157" device="" value="PR"/>
+<part name="SW2" library="MySMD" deviceset="PB157" device="" value="FLASH"/>
 </parts>
 <sheets>
