File: Hardware/SwitchNode Shield/R1/SwitchNode Shield.brd (EAGLE design)
At the start: 96.3 x 44.4 mm, 17 parts

Commit message: Update Mini-Esp and SwitchNode R2
Parts:
- moved U$3 26.5 mm to (20.2, 42.6)
- moved U$1 3.15 mm to (17.8, 56.5)
- moved D1 2.00 mm to (45.2, 45.7)
- moved D3 2.00 mm to (84.5, 45.7)
- moved JP2 2.00 mm to (32.4, 52.5)
- moved R1 2.00 mm to (45.2, 65.4)
- moved R3 2.00 mm to (84.5, 65.4)
- moved S1 2.00 mm to (45.2, 56.5)
- moved S3 2.00 mm to (84.5, 56.5)
- moved U$6 2.00 mm to (31.2, 37.2)
- moved U$7 2.00 mm to (89.4, 37.2)
- moved U$8 2.00 mm to (89.4, 75.7)
- moved U$9 2.00 mm to (31.2, 75.7)
- moved D2 2.00 mm to (64.9, 45.7)
- moved R2 2.00 mm to (64.9, 65.4)
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Other:
- board size 96.3 x 44.4 mm -> 99.3 x 44.4 mm
