File: Hardware/Sandy/R2/Sandy R2.sch (EAGLE design)
At the start: 18 parts, among them SW1 RST, SW2 FLASH

Commit message: Update Sandy R2: + Remove unused resistors and caps + Move 2 buttons to near side to better usability
Parts:
- removed C3: 22nF, SparkFun-Passives:CAP0805
Connections:
- removed net BP: C3.1, RT9013.BP
- net GND: no longer C3.2
Changed lines of the file:
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@@
 <part name="JP2" library="adafruit" deviceset="PINHD-1X9" device=""/>
 <part name="C1" library="SparkFun-Passives" deviceset="CAP" device="0805" value="1uF"/>
-<part name="C3" library="SparkFun-Passives" deviceset="CAP" device="0805" value="22nF"/>
 <part name="C2" library="SparkFun-Capacitors" deviceset="22UF-6.3V-20%(0805)" device="" value="1uF"/>
 <part name="RT9013" library="SparkFun-PowerIC" deviceset="V_REG_MIC5205" device="3.3V" value="3.3V/500mA"/>
@@
 <instance part="JP2" gate="G$1" x="139.7" y="142.24" rot="R180"/>
 <instance part="C1" gate="G$1" x="45.72" y="134.62"/>
-<instance part="C3" gate="G$1" x="81.28" y="137.16"/>
 <instance part="C2" gate="G$1" x="86.36" y="144.78"/>
 <instance part="RT9013" gate="U1" x="68.58" y="147.32"/>
@@
 <pinref part="GND5" gate="1" pin="GND"/>
 <wire x1="86.36" y1="142.24" x2="86.36" y2="134.62" width="0.1524" layer="91"/>
-<pinref part="C3" gate="G$1" pin="2"/>
-<wire x1="81.28" y1="134.62" x2="86.36" y2="134.62" width="0.1524" layer="91"/>
 </segment>
 <segment>
@@
 </segment>
 </net>
-<net name="BP" class="0">
-<segment>
-<pinref part="RT9013" gate="U1" pin="BP"/>
-<pinref part="C3" gate="G$1" pin="1"/>
-<wire x1="76.2" y1="142.24" x2="81.28" y2="142.24" width="0.1524" layer="91"/>
-</segment>
-</net>

Commit message: Update Sandy to move 2 switch buttons near rear side
Parts:
- removed U2: (no value), esp8266modules:ESP12THROUGHOLE
- added U$1: ESP-12-SMD-THIN, My Eagle Lib:ESP-12-SMD-THIN
Connections:
- net A0: now also U$1.ADC; no longer U2.ADC
- net D0: now also U$1.GPIO16; no longer U2.GPIO16
- net D1: now also U$1.GPIO5; no longer U2.GPIO5
- net D2: now also U$1.GPIO4; no longer U2.GPIO4
- net D3: now also U$1.GPIO0; no longer U2.GPIO0
- net D4: now also U$1.GPIO2; no longer U2.GPIO2
- net D5: now also U$1.GPIO14; no longer U2.GPIO14
- net D6: now also U$1.GPIO12; no longer U2.GPIO12
- net D7: now also U$1.GPIO13; no longer U2.GPIO13
- net D8: now also U$1.GPIO15; no longer U2.GPIO15
- net EN: now also U$1.CH_PD; no longer U2.CH_PD
- net GND: now also U$1.GND; no longer U2.GND
- net RST: now also U$1.RESET; no longer U2.RESET
- net RX: now also U$1.RX; no longer U2.RX
- net TX: now also U$1.TX; no longer U2.TX
- net VCC: now also U$1.VCC; no longer U2.VCC
Changed lines of the file:
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@@
 <part name="R1" library="SparkFun-Passives" deviceset="RESISTOR" device="0805-RES" value="100K"/>
 <part name="GND5" library="SparkFun" deviceset="GND" device=""/>
-<part name="U2" library="esp8266modules" deviceset="ESP12" device="THROUGHOLE"/>
 <part name="R5" library="SparkFun-Passives" deviceset="RESISTOR" device="0805-RES" value="10K"/>
 <part name="R6" library="SparkFun-Passives" deviceset="RESISTOR" device="0805-RES" value="10K"/>
@@
 <part name="SW1" library="MySMD" deviceset="PB157" device="" value="RST"/>
 <part name="SW2" library="MySMD" deviceset="PB157" device="" value="FLASH"/>
+<part name="U$1" library="My Eagle Lib" deviceset="ESP-12-SMD-THIN" device=""/>
 </parts>
 <sheets>
@@
 <instance part="R1" gate="G$1" x="55.88" y="137.16" rot="R270"/>
 <instance part="GND5" gate="1" x="86.36" y="132.08"/>
-<instance part="U2" gate="G$1" x="78.74" y="88.9"/>
 <instance part="R5" gate="G$1" x="55.88" y="106.68" rot="R90"/>
 <instance part="R6" gate="G$1" x="48.26" y="106.68" rot="R90"/>
@@
 <instance part="SW1" gate="G$1" x="152.4" y="99.06"/>
 <instance part="SW2" gate="G$1" x="152.4" y="88.9"/>
+<instance part="U$1" gate="G$1" x="78.74" y="86.36"/>
 </instances>
 <busses>
@@
 <wire x1="104.14" y1="81.28" x2="104.14" y2="78.74" width="0.1524" layer="91"/>
 <junction x="104.14" y="78.74"/>
-<pinref part="U2" gate="G$1" pin="GND"/>
+<pinref part="U$1" gate="G$1" pin="GND"/>
 </segment>
 <segment>
@@
 <wire x1="93.98" y1="96.52" x2="106.68" y2="96.52" width="0.1524" layer="91"/>
 <label x="106.68" y="96.52" size="1.778" layer="95"/>
-<pinref part="U2" gate="G$1" pin="TX"/>
+<pinref part="U$1" gate="G$1" pin="TX"/>
 </segment>
 </net>
@@
 <wire x1="93.98" y1="93.98" x2="106.68" y2="93.98" width="0.1524" layer="91"/>
 <label x="106.68" y="93.98" size="1.778" layer="95"/>
-<pinref part="U2" gate="G$1" pin="RX"/>
+<pinref part="U$1" gate="G$1" pin="RX"/>
 </segment>
 </net>
@@
 <wire x1="60.96" y1="96.52" x2="48.26" y2="96.52" width="0.1524" layer="91"/>
 <wire x1="48.26" y1="96.52" x2="48.26" y2="101.6" width="0.1524" layer="91"/>
-<pinref part="U2" gate="G$1" pin="RESET"/>
+<pinref part="U$1" gate="G$1" pin="RESET"/>
 </segment>
 <segment>
@@
 <net name="D2" class="0">
 <segment>
-<pinref part="U2" gate="G$1" pin="GPIO4"/>
 <wire x1="93.98" y1="88.9" x2="106.68" y2="88.9" width="0.1524" layer="91"/>
 <label x="106.68" y="88.9" size="1.778" layer="95"/>
+<pinref part="U$1" gate="G$1" pin="GPIO4"/>
 </segment>
 <segment>
@@
 <net name="D1" class="0">
 <segment>
-<pinref part="U2" gate="G$1" pin="GPIO5"/>
 <wire x1="93.98" y1="91.44" x2="106.68" y2="91.44" width="0.1524" layer="91"/>
 <label x="106.68" y="91.44" size="1.778" layer="95"/>
+<pinref part="U$1" gate="G$1" pin="GPIO5"/>
 </segment>
 <segment>
@@
 <wire x1="93.98" y1="86.36" x2="114.3" y2="86.36" width="0.1524" layer="91"/>
 <label x="106.68" y="86.36" size="1.778" layer="95"/>
-<pinref part="U2" gate="G$1" pin="GPIO0"/>
+<pinref part="U$1" gate="G$1" pin="GPIO0"/>
 </segment>
 <segment>
@@
 <label x="106.68" y="83.82" size="1.778" layer="95"/>
 <pinref part="R3" gate="G$1" pin="1"/>
-<pinref part="U2" gate="G$1" pin="GPIO2"/>
+<pinref part="U$1" gate="G$1" pin="GPIO2"/>
 </segment>
 </net>
@@
 <label x="106.68" y="81.28" size="1.778" layer="95"/>
 <pinref part="R2" gate="G$1" pin="1"/>
-<pinref part="U2" gate="G$1" pin="GPIO15"/>
+<pinref part="U$1" gate="G$1" pin="GPIO15"/>
+<junction x="93.98" y="81.28"/>
+<pinref part="U$1" gate="G$1" pin="GPIO15"/>
 </segment>
 </net>
@@
 <wire x1="60.96" y1="93.98" x2="43.18" y2="93.98" width="0.1524" layer="91"/>
 <label x="43.18" y="93.98" size="1.778" layer="95"/>
-<pinref part="U2" gate="G$1" pin="ADC"/>
+<pinref part="U$1" gate="G$1" pin="ADC"/>
 </segment>
 </net>
@@
 <wire x1="55.88" y1="91.44" x2="55.88" y2="101.6" width="0.1524" layer="91"/>
 <wire x1="60.96" y1="91.44" x2="55.88" y2="91.44" width="0.1524" layer="91"/>
-<pinref part="U2" gate="G$1" pin="CH_PD"/>
+<pinref part="U$1" gate="G$1" pin="CH_PD"/>
 </segment>
 </net>
@@
 <wire x1="60.96" y1="88.9" x2="43.18" y2="88.9" width="0.1524" layer="91"/>
 <label x="43.18" y="88.9" size="1.778" layer="95"/>
-<pinref part="U2" gate="G$1" pin="GPIO16"/>
+<pinref part="U$1" gate="G$1" pin="GPIO16"/>
 </segment>
 </net>
@@
 <wire x1="60.96" y1="86.36" x2="43.18" y2="86.36" width="0.1524" layer="91"/>
 <label x="43.18" y="86.36" size="1.778" layer="95"/>
-<pinref part="U2" gate="G$1" pin="GPIO14"/>
+<pinref part="U$1" gate="G$1" pin="GPIO14"/>
 </segment>
 </net>
@@
 <wire x1="60.96" y1="83.82" x2="43.18" y2="83.82" width="0.1524" layer="91"/>
 <label x="43.18" y="83.82" size="1.778" layer="95"/>
-<pinref part="U2" gate="G$1" pin="GPIO12"/>
+<pinref part="U$1" gate="G$1" pin="GPIO12"/>
 </segment>
 </net>
@@
 <wire x1="60.96" y1="81.28" x2="43.18" y2="81.28" width="0.1524" layer="91"/>
 <label x="43.18" y="81.28" size="1.778" layer="95"/>
-<pinref part="U2" gate="G$1" pin="GPIO13"/>
+<pinref part="U$1" gate="G$1" pin="GPIO13"/>
 </segment>
 </net>
@@
 <segment>
 <wire x1="60.96" y1="78.74" x2="45.72" y2="78.74" width="0.1524" layer="91"/>
-<pinref part="U2" gate="G$1" pin="VCC"/>
 <pinref part="VCC" gate="G$1" pin="VCC"/>
-</segment>
-<segment>
+<pinref part="U$1" gate="G$1" pin="VCC"/>
+</segment>
+<segment>
