File: Hardware/Ivy Sensor Shield/Ivy Sensor Shield.brd (EAGLE design)
At the start: 50.8 x 41.3 mm, 28 parts, among them IC2 MCP73831/OT

Commit message: Update Ivy Sensor to use locked pad version of Sandy Esp
Parts:
- U$2: value MINI-ESP -> MINI-ESPMINI-ESP-LOCK; device My Eagle Lib:MINI-ESP -> My Eagle Lib:MINI-ESP-LOCK
