File: Hardware/Ivy Sensor Shield/Ivy Sensor Shield.sch (EAGLE design)
At the start: 24 parts, among them IC2 MCP73831/OT

Commit message: Update Ivy Sensor to use locked pad version of Sandy Esp
Parts:
- U$2: value MINI-ESP -> MINI-ESPMINI-ESP-LOCK; device My Eagle Lib:MINI-ESP -> My Eagle Lib:MINI-ESPMINI-ESP-LOCK
Changed lines of the file:
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@@
 </classes>
 <parts>
-<part name="U$2" library="My Eagle Lib" deviceset="MINI-ESP" device=""/>
+<part name="U$2" library="My Eagle Lib" deviceset="MINI-ESP" device="MINI-ESP-LOCK" value="MINI-ESPMINI-ESP-LOCK"/>
 <part name="JP1" library="adafruit" deviceset="PINHD-1X9" device=""/>
 <part name="JP3" library="adafruit" deviceset="PINHD-1X9" device=""/>
