File: Hardware/Kodi Remote/R2/Kodi Remote.sch (EAGLE design)
At the start: 17 parts

Commit message: Minor change to Kodi Remote
Connections:
- net A1 renamed A0
- net RST1 renamed RST
- net RX1 renamed RX
- net TX1 renamed TX
- removed net GND1: U$10.GND
- net GND: now also U$10.GND
Changed lines of the file:
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@@
 <pinref part="GND9" gate="1" pin="GND"/>
+</segment>
+<segment>
+<pinref part="U$10" gate="G$1" pin="GND"/>
+<wire x1="172.72" y1="48.26" x2="177.8" y2="48.26" width="0.1524" layer="91"/>
 </segment>
 </net>
@@
 </segment>
 </net>
-<net name="GND1" class="0">
-<segment>
-<pinref part="U$10" gate="G$1" pin="GND"/>
-<wire x1="172.72" y1="48.26" x2="177.8" y2="48.26" width="0.1524" layer="91"/>
-</segment>
-</net>
 <net name="5V" class="0">
 <segment>
@@
 </segment>
 </net>
-<net name="A1" class="0">
+<net name="A0" class="0">
 <segment>
 <pinref part="U$10" gate="G$1" pin="A0"/>
@@
 </segment>
 </net>
-<net name="RST1" class="0">
+<net name="RST" class="0">
 <segment>
 <pinref part="U$10" gate="G$1" pin="RST"/>
@@
 </segment>
 </net>
-<net name="TX1" class="0">
+<net name="TX" class="0">
 <segment>
 <pinref part="U$10" gate="G$1" pin="TX"/>
@@
 </segment>
 </net>
-<net name="RX1" class="0">
+<net name="RX" class="0">
 <segment>
 <pinref part="U$10" gate="G$1" pin="RX"/>
