File: Hardware/Ivy Sensor Shield/R2/Ivy Sensor Shield.sch (EAGLE design)
At the start: 12 parts

Commit message: Correct wiring for Ivy Sensor Shield.brd
Parts:
- renumbered MQ_2 to RSV
Connections:
- net AOUT renamed NC2
- removed net VIN: PIR.1, RSV.1
- net 5V: now also PIR.1, RSV.1
